File: SensorBracelet/KiCad/OM-EPSC3-Micro.kicad_pcb (KiCad board)
At the start: 2 copper layers, 27.5 x 52 mm, 23 parts, among them J1 Conn_01x04_Pin, J2 Conn_01x02_Pin, J3 Conn_01x02_Pin, J4 JST_02, J5 Conn_01x01_Pin, SW2 SW_Push, U2 LTC4054ES5-4.2, U5 TPS7A03

Commit message: Lask V2
Parts:
- removed J1: Conn_01x04_Pin, Connector_PinHeader_2.54mm:PinHeader_1x04_P2.54mm_Vertical
- removed J5: Conn_01x01_Pin, Connector_PinHeader_2.54mm:PinHeader_1x01_P2.54mm_Vertical
- added J6: Conn_01x05_Pin, Connector_PinHeader_1.27mm:PinHeader_1x05_P1.27mm_Vertical, F.Cu at (217.2, 135.5)
- moved SW2 0.26 mm to (229.0, 138.8)
- moved J3 0.25 mm to (234.4, 134.6)
Routing:
- net +3V3: track 90.8 -> 27.0 mm, vias 2 -> 3
- net LDO_EN: track 42.1 -> 67.9 mm, vias 2 -> 0
- net Net-(MAX1-CLEAR): track 20.8 -> 6.83 mm
- net +5V: track 72.8 -> 62.6 mm, vias 1 -> 2
- net GND: track 25.1 -> 15.3 mm
- net +3V8: track 76.3 -> 67.8 mm, vias 2 -> 1
- net ADC3: track 38.7 -> 45.0 mm
- net RMT-BTN: track 38.0 -> 36.0 mm
- net hall_0: track 26.6 -> 28.5 mm
- net hall_1: track 40.7 -> 41.8 mm
- net ADC2: track 26.8 -> 25.8 mm, vias 1 -> 0
- net (no net): vias 1 -> 0
