File: SensorBracelet/KiCad/OM-EPSC3-Micro.kicad_sch (KiCad schematic)
At the start: 23 parts, among them J1 Conn_01x04_Pin, J2 Conn_01x02_Pin, J3 Conn_01x02_Pin, J4 JST_02, J5 Conn_01x01_Pin, SW1 SW_Push, U2 LTC4054ES5-4.2, U2 TPS7A03

Commit message: Lask V2
Parts:
- removed J1: Conn_01x04_Pin, Connector_PinHeader_2.54mm:PinHeader_1x04_P2.54mm_Vertical, symbol Connector:Conn_01x04_Pin
- removed J5: Conn_01x01_Pin, Connector_PinHeader_2.54mm:PinHeader_1x01_P2.54mm_Vertical, symbol Connector:Conn_01x01_Pin
- added J6: Conn_01x05_Pin, Connector_PinHeader_1.27mm:PinHeader_1x05_P1.27mm_Vertical, symbol Connector:Conn_01x05_Pin
Connections:
- net +3V3: now also J6.2 (Pin_2)
- net +5V: now also J6.1 (Pin_1)
- net ADC2: now also J6.4 (Pin_4)
- net ADC3: now also J6.3 (Pin_3)
- net GND: now also J6.5 (Pin_5)
Changed lines of the file:
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@@
+    (stroke (width 0) (type default))
+  )
+  (wire (pts (xy 132.08 93.98) (xy 119.38 93.98))
     (stroke (width 0) (type default))
   )
@@
     )
   )
-  (symbol (lib_id "Connector:Conn_01x04_Pin") (at 114.3 99.06 0) (unit 1)
-    (in_bom yes) (on_board yes) (dnp no) (fields_autoplaced)
-    (property "Reference" "J1" (at 114.935 91.44 0)
-      (effects (font (size 1.27 1.27)))
-    )
-    (property "Value" "Conn_01x04_Pin" (at 114.935 93.98 0)
-      (effects (font (size 1.27 1.27)))
-    )
-    (property "Footprint" "Connector_PinHeader_2.54mm:PinHeader_1x04_P2.54mm_Vertical" (at 114.3 99.06 0)
-      (effects (font (size 1.27 1.27)) hide)
-    )
-    (property "Datasheet" "~" (at 114.3 99.06 0)
-      (effects (font (size 1.27 1.27)) hide)
-    )
-    (pin "1")
-    (pin "2")
-    (pin "3")
-    (pin "4")
-    (instances
-      (project "OM-EPSC3-Micro"
-        (path "/c7fe26ae-9505-4931-9cd8-090fc73447cd"
-          (reference "J1") (unit 1)
-        )
-      )
-    )
-  )
   (symbol (lib_id "Sensor_Current:A1369xUA-10") (at 120.65 40.64 0) (unit 1)
     (in_bom yes) (on_board yes) (dnp no)
@@
     )
   )
-  (symbol (lib_id "power:+5V") (at 101.6 101.6 0) (unit 1)
-    (in_bom yes) (on_board yes) (dnp no) (fields_autoplaced)
-    (property "Reference" "#PWR020" (at 101.6 105.41 0)
-      (effects (font (size 1.27 1.27)) hide)
-    )
-    (property "Value" "+5V" (at 101.6 96.52 0)
-      (effects (font (size 1.27 1.27)))
-    )
-    (property "Footprint" "" (at 101.6 101.6 0)
-      (effects (font (size 1.27 1.27)) hide)
-    )
-    (property "Datasheet" "" (at 101.6 101.6 0)
-      (effects (font (size 1.27 1.27)) hide)
-    )
-    (pin "1")
-    (instances
-      (project "OM-EPSC3-Micro"
-        (path "/c7fe26ae-9505-4931-9cd8-090fc73447cd"
-          (reference "#PWR020") (unit 1)
-        )
-      )
-    )
-  )
   (symbol (lib_id "power:+3V8") (at 177.8 129.54 0) (unit 1)
     (in_bom yes) (on_board yes) (dnp no) (fields_autoplaced)
@@
         (path "/c7fe26ae-9505-4931-9cd8-090fc73447cd"
           (reference "#PWR045") (unit 1)
+        )
+      )
+    )
+  )
+  (symbol (lib_id "Connector:Conn_01x05_Pin") (at 114.3 99.06 0) (unit 1)
+    (in_bom yes) (on_board yes) (dnp no)
+    (property "Reference" "J6" (at 114.935 88.9 0)
+      (effects (font (size 1.27 1.27)))
+    )
+    (property "Value" "Conn_01x05_Pin" (at 111.76 99.06 90)
+      (effects (font (size 1.27 1.27)))
+    )
+    (property "Footprint" "Connector_PinHeader_1.27mm:PinHeader_1x05_P1.27mm_Vertical" (at 114.3 99.06 0)
+      (effects (font (size 1.27 1.27)) hide)
+    )
+    (property "Datasheet" "~" (at 114.3 99.06 0)
+      (effects (font (size 1.27 1.27)) hide)
+    )
+    (pin "1")
+    (pin "2")
+    (pin "3")
+    (pin "4")
+    (pin "5")
+    (instances
+      (project "OM-EPSC3-Micro"
+        (path "/c7fe26ae-9505-4931-9cd8-090fc73447cd"
+          (reference "J6") (unit 1)
         )
       )
@@
     )
   )
+  (symbol (lib_id "power:+5V") (at 132.08 93.98 0) (unit 1)
+    (in_bom yes) (on_board yes) (dnp no) (fields_autoplaced)
+    (property "Reference" "#PWR021" (at 132.08 97.79 0)
+      (effects (font (size 1.27 1.27)) hide)
+    )
+    (property "Value" "+5V" (at 132.08 88.9 0)
+      (effects (font (size 1.27 1.27)))
+    )
+    (property "Footprint" "" (at 132.08 93.98 0)
+      (effects (font (size 1.27 1.27)) hide)
+    )
+    (property "Datasheet" "" (at 132.08 93.98 0)
+      (effects (font (size 1.27 1.27)) hide)
+    )
+    (pin "1")
+    (instances
+      (project "OM-EPSC3-Micro"
+        (path "/c7fe26ae-9505-4931-9cd8-090fc73447cd"
+          (reference "#PWR021") (unit 1)
+        )
+      )
+      (project "ThinkTankTimerVote"
+        (path "/f5106d17-538e-4380-9554-aa558f4a587a"
+          (reference "#PWR013") (unit 1)
+        )
+      )
+    )
+  )
   (symbol (lib_id "Jumper:SolderJumper_2_Open") (at 139.7 33.02 0) (unit 1)
     (in_bom yes) (on_board yes) (dnp no) (fields_autoplaced)
@@
         )
       )
-    )
-  )
-  (symbol (lib_id "Connector:Conn_01x01_Pin") (at 96.52 101.6 0) (unit 1)
-    (in_bom yes) (on_board yes) (dnp no) (fields_autoplaced)
-    (property "Reference" "J5" (at 97.155 96.52 0)
-      (effects (font (size 1.27 1.27)))
-    )
-    (property "Value" "Conn_01x01_Pin" (at 97.155 99.06 0)
-      (effects (font (size 1.27 1.27)))
-    )
-    (property "Footprint" "Connector_PinHeader_2.54mm:PinHeader_1x01_P2.54mm_Vertical" (at 96.52 101.6 0)
-      (effects (font (size 1.27 1.27)) hide)
-    )
-    (property "Datasheet" "~" (at 96.52 101.6 0)
-      (effects (font (size 1.27 1.27)) hide)
-    )
-    (pin "1")
-    (instances
-      (project "OM-EPSC3-Micro"
-        (path "/c7fe26ae-9505-4931-9cd8-090fc73447cd"
-          (reference "J5") (unit 1)
-        )
-      )
