File: Labeler/KiCad/LASK_V2-0/LASK-V2-0.kicad_pcb (KiCad board)
At the start: 4 copper layers, 75 x 35 mm, 45 parts, among them J1 Conn_01x04, J2 JST_02, J3 Conn_01x10_Pin, J6 Conn_01x07_Pin, J9 Conn_01x04, P1 USB_C_Plug_USB2.0, Q2 VP0610T, U2 ESP32-S3-WROOM-1-N16R8, U3 TPS7A03, U4 LTC4054ES5-4.2

Commit message: LASK5-V2.1
Parts:
- removed P1: USB_C_Plug_USB2.0, Connector_USB:USB_C_Receptacle_GCT_USB4085
- added J4: USB_C_Receptacle, Connector_USB:USB_C_Receptacle_HRO_TYPE-C-31-M-12, F.Cu at (151.9, 98.4)
- JP1: moved to B.Cu
- moved JP1 14.5 mm to (161.1, 81.9), turned to 180 degrees
- moved D2 5.08 mm to (160.7, 73.3)
- moved R8 3.18 mm to (164.3, 82.2)
- moved R7 2.53 mm to (158.0, 81.5), turned to -90 degrees
- moved R1 2.53 mm to (165.2, 92.3), turned to 0 degrees
- moved R5 2.33 mm to (166.4, 73.0)
- moved U4 2.19 mm to (160.7, 77.5)
- moved R9 2.05 mm to (152.5, 69.6), turned to 180 degrees
- moved C7 1.87 mm to (149.2, 73.3)
- moved C5 1.17 mm to (133.9, 94.3), turned to -90 degrees
- moved R6 0.85 mm to (138.1, 94.0)
- moved R2 0.77 mm to (164.9, 94.1), turned to 0 degrees
- moved Q2 0.74 mm to (155.8, 73.6)
- moved C1 0.69 mm to (163.9, 70.7)
- moved U3 0.36 mm to (153.0, 78.0)
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Connections:
- J3 pad 10: GP42 -> TX
- J3 pad 3: GP21 -> GP13
- J3 pad 4: GP18 -> GP14
- J3 pad 5: GP17 -> GP21
- J3 pad 6: GP34 -> GP33
- J3 pad 7: GP33 -> GP34
- J3 pad 8: TX -> GP42
- J6 pad 3: GP16 -> GP15
- J6 pad 4: GP15 -> GP16
- J6 pad 5: GP14 -> GP17
- J6 pad 6: GP13 -> GP18
Routing:
- net b_select: track 87.6 -> 36.3 mm, vias 3 -> 2
- net hall_3: track 72.3 -> 97.2 mm, vias 1 -> 0
- net GP18: track 47.4 -> 23.1 mm, vias 3 -> 1
- net ADC_BAT: track 22.9 -> 46.0 mm, vias 1 -> 2
- net GP42: track 76.4 -> 53.8 mm, vias 2 -> 1
- net 100: track 58.2 -> 37.2 mm
- net GP17: track 44.6 -> 23.8 mm, vias 2 -> 1
- net D+: track 17.0 -> 35.4 mm, vias 1 -> 2
- net Net-(JP1-A): track 26.6 -> 8.84 mm
- net GP14: track 17.4 -> 33.0 mm
- net VIN: track 43.3 -> 28.0 mm
- net GP33: track 61.3 -> 47.5 mm, vias 2 -> 1
- net D-: track 19.9 -> 33.1 mm, vias 1 -> 2
- net SCL: track 63.8 -> 77.0 mm, vias 2 -> 3
- net JSW: track 67.0 -> 78.9 mm, vias 2 -> 1
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
Commit message: LASK5-V2.1 Updates
Routing:
- net D+: track 35.4 -> 17.6 mm, vias 2 -> 0
- net D-: track 33.1 -> 17.0 mm, vias 2 -> 0
- net VBUS: track 75.5 -> 69.7 mm, vias 8 -> 7
- net Net-(J4-CC1): track 20.0 -> 16.0 mm
- net Net-(J4-CC2): track 16.9 -> 18.4 mm
- net b_start: track 34.1 -> 35.4 mm
- net b_select: track 36.3 -> 37.5 mm
