File: Labeler/KiCad/LASK_V2-0/LASK-V2-0.kicad_sch (KiCad schematic)
At the start: 45 parts, among them J3 Conn_01x10_Pin, J4 Conn_01x04, J4 JST_02, J6 Conn_01x07_Pin, P1 USB_C_Plug_USB2.0, Q2 VP0610T, SW1 SW_Push, U2 ESP32-S3-WROOM-1-N16R8, U2 LTC4054ES5-4.2, U2 TPS7A03

Commit message: LASK5-V2.1
Parts:
- removed P1: USB_C_Plug_USB2.0, Connector_USB:USB_C_Receptacle_GCT_USB4085, symbol Connector:USB_C_Plug_USB2.0
- removed R8 (x2): 5.1K, Resistor_SMD:R_0603_1608Metric, symbol Device:R
- added J4: USB_C_Receptacle, Connector_USB:USB_C_Receptacle_HRO_TYPE-C-31-M-12, symbol Connector:USB_C_Receptacle
- added R8 (x2): 5.1K, Resistor_SMD:R_0603_1608Metric, symbol Device:R
Connections:
- net D+: now also J4.A6 (D+), J4.B6 (D+)
- net D-: now also J4.A7 (D-), J4.B7 (D-)
- net GND: now also J4.A1 (GND), J4.A12 (GND), J4.B1 (GND), J4.B12 (GND), J4.S1 (SHIELD), R8.2, R8.2
- net GP13: now also J3.3 (Pin_3); no longer J6.6 (Pin_6)
- net GP14: now also J3.4 (Pin_4); no longer J6.5 (Pin_5)
- net GP15: now also J6.3 (Pin_3); no longer J6.4 (Pin_4)
- net GP16: now also J6.4 (Pin_4); no longer J6.3 (Pin_3)
- net GP17: now also J6.5 (Pin_5); no longer J3.5 (Pin_5)
- net GP18: now also J6.6 (Pin_6); no longer J3.4 (Pin_4)
- net GP21: now also J3.5 (Pin_5); no longer J3.3 (Pin_3)
- net GP33: now also J3.6 (Pin_6); no longer J3.7 (Pin_7)
- net GP34: now also J3.7 (Pin_7); no longer J3.6 (Pin_6)
- net GP42: now also J3.8 (Pin_8); no longer J3.10 (Pin_10)
- net TX: now also J3.10 (Pin_10); no longer J3.8 (Pin_8)
- net VBUS: now also J4.A4 (VBUS), J4.A9 (VBUS), J4.B4 (VBUS), J4.B9 (VBUS)
- new net: J4.B5 (CC2), R8.1
- new net: J4.A5 (CC1), R8.1

Commit message: LASK5 V2 Hardware Update
Working PCB for LASK5 V2
Parts:
- D2: value LED GREEN -> CHRG LED
- renumbered J4 to BattExtLTC4054, C15 to C1, C15 to C2, C15 to C3, C15 to C4, C15 to C5, C4 to C6, C3 to C7, C9 to C8, H0 to H2, H1 to H3, H0 to H4, J4 to J1, J4 to J2, J4 to J9, R8 to R1, R8 to R2, R1 to R3, R8 to R4, R9 to R5, R8 to R6, R8 to R7, R1 to R9, SW1 to SW_PWR1, U2 to U3, U2 to U4
Other:
- moved on the sheet: BattExtLTC4054, C6, C7, C8, D1, D2, J2, J4, JP1, MAX1, Q2, R1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
