File: Labeler/KiCad/LASK_V3-0/LASK5-V3-0.kicad_pcb (KiCad board)
At the start: 4 copper layers, 75 x 35 mm, 45 parts, among them J1 Conn_01x04, J2 JST_02, J3 Conn_01x10_Pin, J4 USB_C_Receptacle, J6 Conn_01x07_Pin, J9 Conn_01x04, Q2 VP0610T, U2 ESP32-S3-WROOM-1-N16R8, U3 TPS7A03, U4 LTC4054ES5-4.2

Commit message: LASK5 V3 and OM-FlexGrid
Parts:
- added C10: 0.1 uF, Capacitor_SMD:C_0603_1608Metric, F.Cu at (153.5, 85.8)
- added C11: 2.2 uF, Capacitor_SMD:C_0603_1608Metric, F.Cu at (156.8, 84.0)
- added C9: 100 uF, Capacitor_SMD:C_0603_1608Metric, F.Cu at (168.0, 87.7)
- added D3: BAT54C, Package_TO_SOT_SMD:SOT-23, F.Cu at (174.5, 70.6)
- added D4: 1N4007, Diode_SMD:D_SOD-123, F.Cu at (170.0, 87.3)
- added IC1: ICM-42688-P, ICM-42688-P:IIM42352, F.Cu at (156.5, 86.8)
- added J5: Conn_01x02, Connector_PinHeader_2.00mm:PinHeader_1x02_P2.00mm_Vertical, F.Cu at (165.5, 88.0)
- added Q1: IRLML2060, Package_TO_SOT_SMD:SOT-23, F.Cu at (161.9, 90.0)
- added Q3: IRLML2060, Package_TO_SOT_SMD:SOT-23, F.Cu at (174.6, 78.0)
- added R10: 10k, Resistor_SMD:R_0603_1608Metric, F.Cu at (150.2, 81.9)
- added R11: 10k, Resistor_SMD:R_0603_1608Metric, F.Cu at (150.2, 85.0)
- D2: value LED GREEN -> CHRG LED
- J3: value Conn_01x10_Pin -> Conn_01x04_Pin; footprint Connector_PinHeader_2.00mm:PinHeader_1x10_P2.00mm_Vertical -> Connector_PinHeader_2.00mm:PinHeader_1x04_P2.00mm_Vertical
- J6: value Conn_01x07_Pin -> Conn_01x06_Pin; footprint Connector_PinHeader_2.00mm:PinHeader_1x07_P2.00mm_Vertical -> Connector_PinHeader_1.27mm:PinHeader_1x06_P1.27mm_Vertical; moved to B.Cu
- moved J6 21.9 mm to (133.7, 70.7), turned to -90 degrees
- moved J3 14.8 mm to (146.5, 89.0)
- moved D1 3.17 mm to (169.4, 68.5)
- moved R2 1.77 mm to (166.7, 94.1)
- moved R1 1.51 mm to (166.7, 92.3)
- moved D2 0.50 mm to (160.6, 73.8)
- renumbered J9 to J1, J1 to J9
Connections:
- net b_select renamed SELECT
- J3 pad 3: GP13 -> GP15
- J3 pad 4: GP14 -> GP16
- J6 pad 1: GND -> +3V3
- J6 pad 2: +3V3 -> SPI_MISO
- J6 pad 3: GP15 -> SPI_SCK
- J6 pad 4: GP16 -> SPI_MOSI
- J6 pad 5: GP17 -> CS
- J6 pad 6: GP18 -> GND
- J9 pad 1: GND -> +3V3
- J9 pad 2: +3V3 -> GND
- SW_M1 pad 1: b_start -> MENU
- U2 pad 10: GP17 -> MOT_SIG
- U2 pad 11: GP18 -> ADC_BAT
- U2 pad 19: b_start -> SPI_MISO
- U2 pad 20: ADC_BAT -> SPI_SCK
- U2 pad 21: GP13 -> SPI_MOSI
- U2 pad 22: GP14 -> CS
- U2 pad 23: GP21 -> MENU
- U2 pad 26: unconnected-(U2-IO45-Pad26) -> PWR_OFF
- U2 pad 35: GP42 -> unconnected-(U2-IO42-Pad35)
- U3 pad 3: LDO_EN -> Net-(U3-EN)
Routing:
- net TX: track 61.8 -> 0.00 mm, vias 1 -> 0
- net RX: track 58.3 -> 0.00 mm, vias 1 -> 0
- net GP42: track 53.8 -> 0.00 mm, vias 1 -> 0
- net MENU: track 0.00 -> 47.1 mm, vias 0 -> 4
- net PWR_OFF: track 0.00 -> 46.1 mm, vias 0 -> 2
- net SPI_MISO: track 0.00 -> 45.2 mm, vias 0 -> 2
- net GND: track 83.5 -> 127.8 mm, vias 11 -> 15
- net CS: track 0.00 -> 41.1 mm, vias 0 -> 1
- net SPI_SCK: track 0.00 -> 40.0 mm, vias 0 -> 2
- net SPI_MOSI: track 0.00 -> 38.3 mm, vias 0 -> 2
- net GP21: track 36.0 -> 0.00 mm, vias 1 -> 0
- net b_start: track 35.4 -> 0.00 mm, vias 2 -> 0
- net GP14: track 33.0 -> 0.00 mm, vias 1 -> 0
- net GP13: track 30.5 -> 0.00 mm, vias 1 -> 0
- net Net-(U3-EN): track 0.00 -> 28.4 mm, vias 0 -> 2
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