File: Labeler/KiCad/LASK_V3-0/LASK5-V3-0.kicad_sch (KiCad schematic)
At the start: 46 parts, among them J1 Conn_01x04, J2 JST_02, J3 Conn_01x10_Pin, J4 USB_C_Receptacle, J6 Conn_01x07_Pin, J9 Conn_01x04, Q2 VP0610T, U2 ESP32-S3-WROOM-1-N16R8, U3 TPS7A03, U4 LTC4054ES5-4.2

Commit message: LASK5 V3 and OM-FlexGrid
Parts:
- removed J3: Conn_01x10_Pin, Connector_PinHeader_2.00mm:PinHeader_1x10_P2.00mm_Vertical, symbol Connector:Conn_01x10_Pin
- removed J6: Conn_01x07_Pin, Connector_PinHeader_2.00mm:PinHeader_1x07_P2.00mm_Vertical, symbol Connector:Conn_01x07_Pin
- added C10: 0.1 uF, Capacitor_SMD:C_0603_1608Metric, symbol Device:C
- added C11: 2.2 uF, Capacitor_SMD:C_0603_1608Metric, symbol Device:C
- added C9: 100 uF, Capacitor_SMD:C_0603_1608Metric, symbol Device:C
- added D4: 1N4007, Diode_SMD:D_SOD-123, symbol Diode:1N4007
- added IC1: ICM-42688-P, IIM42352, symbol ICM-42688-P:ICM-42688-P
- added J3: Conn_01x04_Pin, Connector_PinHeader_2.00mm:PinHeader_1x04_P2.00mm_Vertical, symbol Connector:Conn_01x04_Pin
- added J5: Conn_01x02, Connector_PinHeader_2.00mm:PinHeader_1x02_P2.00mm_Vertical, symbol Connector_Generic:Conn_01x02
- added J6: Conn_01x06_Pin, Connector_PinHeader_1.27mm:PinHeader_1x06_P1.27mm_Vertical, symbol Connector:Conn_01x06_Pin
- added Q1, Q3: IRLML2060, Package_TO_SOT_SMD:SOT-23, symbol Transistor_FET:IRLML2060
- added R10, R11: 10k, Resistor_SMD:R_0603_1608Metric, symbol Device:R
- renumbered J9 to J1, J1 to J9
Connections:
- net GP18 is gone; now on net ADC_BAT: U2.11 (IO18)
- net +3V3: now also J9.1 (Pin_1), C10.1, C11.1, IC1.5 (VDDIO), IC1.8 (VDD), J3.2 (Pin_2), J6.1 (Pin_1); no longer J9.2 (Pin_2)
- net ADC_BAT: no longer U2.20 (IO12)
- net GND: now also J9.2 (Pin_2), C10.2, C11.2, IC1.11 (RESV_5), IC1.6 (GND), IC1.7 (RESV_3), J3.1 (Pin_1), J6.6 (Pin_6), Q1.2 (S), Q3.2 (S), R11.1; no longer J9.1 (Pin_1)
- net GP15: now also J3.3 (Pin_3)
- net GP16: now also J3.4 (Pin_4)
- net GP33: now also IC1.4 (INT1/INT)
- net GP34: now also IC1.9 (INT2/FSYNC/CLKIN)
- net SCL: now also IC1.13 (SCL/SCLK)
- net SDA: now also IC1.14 (SDA/SDIO/ASDI)
- net at MAX1.1 (In), SW_PWR1.2: now also Q3.3 (D)
- net PWR_OFF: now reaches U2.26 (IO45)
- net PWR_OFF: now also Q3.1 (G)
- net GP13 renamed SPI_MOSI
- net SPI_MOSI: now also J6.4 (Pin_4)
- net GP14 renamed CS
- net CS: now also J6.5 (Pin_5)
- net GP17 renamed MOT_SIG
- net MOT_SIG: now also R10.2
- net GP21 renamed MENU
- net MENU: now also SW_M1.1
- net GP42: no longer names the net of U2.35 (IO42)
- net b_select renamed SELECT
- net b_start renamed SPI_MISO
- net SPI_MISO: now also J6.2 (Pin_2); no longer SW_M1.1
- new net: Q1.1 (G), R10.1, R11.2
- new net Batt+: C9.2, D4.1 (K), J5.1 (Pin_1)
- new net MotorGND: C9.1, D4.2 (A), J5.2 (Pin_2), Q1.3 (D)
- new net SPI_SCK: J6.3 (Pin_3), U2.20 (IO12)
Other:
- note added: "ESP32-S3 WROOM-1 N16R8"
- note added: "Haptic Motor"
- note added: "SPI(1) SCK=12, MOSI=11, MISO=13"
- note added: "TODO: Put ESD Protection Check GPIOs for Conflicts Add decoupling Capacitors"
- note added: "TPS7A0333 LDO with EN 3.3V"
- note added: "VBUS_OR_VBAT"
- note removed: "ESP32-S3 Supermini"
- note removed: "TPS7A0333 LDO with EN 3.3v!"
- moved on the sheet: BattExtLTC4054, J2, MAX1, R3, SW_PWR1
